File: Kicad files/keyboardepi pico.kicad_pcb (KiCad board)
At the start: 2 copper layers, 299.8 x 97 mm, 141 parts, among them U1 Raspberry_Pi_Pico

Commit message: Updated the PCB
Routing:
- net row0: track 300.0 -> 298.1 mm
- net row2: track 254.1 -> 252.2 mm
- net row1: track 255.8 -> 254.0 mm
- net gnd: track 565.2 -> 563.6 mm
- net Net-(D8-A): track 9.60 -> 8.31 mm
- net Net-(D121-A): track 4.96 -> 3.98 mm
- net row4: track 294.0 -> 293.0 mm
- net col11: track 170.5 -> 169.6 mm
- net Net-(D58-A): track 4.28 -> 3.55 mm

Commit message: finalizing the project for shipping
Parts:
- D1, D10, D11, D12, D120, D121, D13, D15, D16, D18, D19, D2, D20, D21, D22, D23, D24, D25, D26, D27, D28, D3, D30, D31, D33, D34, D35, D36, D37, D38, D39, D4, D40, D41, D42, D43, D45, D46, D48, D49, D5, D50, D51, D52, D53, D54, D55, D56, D57, D58, D6, D60, D61, D62, D63, D68, D7, D73, D74, D75, D8, D9: moved to B.Cu
Routing:
- net row3: track 436.0 -> 334.7 mm, vias 4 -> 2
- net row2: track 252.2 -> 263.6 mm, vias 2 -> 25
- net row4: track 293.0 -> 299.5 mm, vias 2 -> 7
- net row1: track 254.0 -> 260.2 mm, vias 8 -> 31
- net col12: track 230.8 -> 234.7 mm
- net col1: track 332.8 -> 336.7 mm
- net col9: track 203.2 -> 199.6 mm
- net col11: track 169.6 -> 172.9 mm
- net Net-(D9-A): track 10.8 -> 8.02 mm, vias 1 -> 0
- net row0: track 298.1 -> 295.5 mm, vias 12 -> 28
- net col2: track 351.1 -> 352.8 mm
- net Net-(D68-A): track 5.17 -> 3.61 mm, vias 1 -> 0
- net Net-(D6-A): track 8.07 -> 8.99 mm, vias 1 -> 2
- net col4: track 350.3 -> 350.9 mm
- net col14: track 148.4 -> 149.0 mm
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
Commit message: Removed the LEDs
Parts:
- removed D14, D17, D29, D32, D44, D47, D59, D64, D65, D66, D67: WS2812B, LED_SMD:LED_WS2812B_PLCC4_5.0x5.0mm_P3.2mm
Connections:
- U1 pad 28: gnd -> unconnected-(U1-GND-Pad28)
- U1 pad 29: data in led -> unconnected-(U1-GPIO22-Pad29)
- U1 pad 40: 5v -> unconnected-(U1-VBUS-Pad40)
Routing:
- net 5v: track 593.5 -> 0.00 mm, vias 10 -> 0
- net gnd: track 563.8 -> 0.01 mm, vias 9 -> 0
- net data in led: track 266.5 -> 0.00 mm, vias 5 -> 0
- net Net-(D59-DOUT): track 252.9 -> 0.00 mm, vias 2 -> 0
- net Net-(D65-DOUT): track 42.9 -> 0.00 mm
- net Net-(D64-DOUT): track 42.6 -> 0.00 mm
- net Net-(D14-DOUT): track 33.5 -> 0.00 mm
- net Net-(D44-DOUT): track 32.9 -> 0.00 mm, vias 2 -> 0
- net Net-(D32-DOUT): track 32.5 -> 0.00 mm
- net Net-(D29-DOUT): track 32.3 -> 0.00 mm, vias 2 -> 0
- net Net-(D17-DOUT): track 32.0 -> 0.00 mm
- net Net-(D47-DOUT): track 28.5 -> 0.00 mm
- net unconnected-(U1-GND-Pad28): track 0.00 -> 22.9 mm
- net col2: track 352.8 -> 333.1 mm
- net col8: track 224.3 -> 214.0 mm
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
Commit message: fixing the PCB
Parts:
- moved U1 2.37 mm to (280.9, 37.8)
Routing:
- net col10: track 248.8 -> 189.2 mm, vias 1 -> 2
- net unconnected-(U1-GND-Pad13): track 0.00 -> 43.9 mm
- net col13: track 160.6 -> 126.3 mm, vias 5 -> 4
- net col3: track 296.2 -> 270.8 mm, vias 1 -> 3
- net unconnected-(U1-GND-Pad28): track 22.9 -> 0.00 mm
- net col7: track 257.7 -> 276.4 mm
- net col2: track 333.1 -> 319.1 mm
- net col0: track 352.7 -> 344.5 mm, vias 2 -> 1
- net col12: track 234.7 -> 238.6 mm, vias 4 -> 8
- net col4: track 350.9 -> 353.5 mm, vias 1 -> 6
- net col1: track 336.7 -> 339.2 mm
- net col14: track 149.0 -> 151.5 mm, vias 1 -> 4
- net col8: track 214.0 -> 216.2 mm
- net col5: track 305.9 -> 307.8 mm, vias 1 -> 4
- net col11: track 172.9 -> 171.3 mm, vias 1 -> 5
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
Commit message: finishing up to ship the project
Parts:
- added D14: WS2812B, LED_SMD:LED_WS2812B_PLCC4_5.0x5.0mm_P3.2mm, B.Cu at (30.3, 13.0)
- added D17: WS2812B, LED_SMD:LED_WS2812B_PLCC4_5.0x5.0mm_P3.2mm, B.Cu at (54.2, 13.1)
- added D29: WS2812B, LED_SMD:LED_WS2812B_PLCC4_5.0x5.0mm_P3.2mm, B.Cu at (74.3, 13.1)
- added D32: WS2812B, LED_SMD:LED_WS2812B_PLCC4_5.0x5.0mm_P3.2mm, B.Cu at (100.1, 13.2)
- added D44: WS2812B, LED_SMD:LED_WS2812B_PLCC4_5.0x5.0mm_P3.2mm, B.Cu at (124.5, 13.1)
- added D47: WS2812B, LED_SMD:LED_WS2812B_PLCC4_5.0x5.0mm_P3.2mm, B.Cu at (151.7, 13.1)
- added D59: WS2812B, LED_SMD:LED_WS2812B_PLCC4_5.0x5.0mm_P3.2mm, B.Cu at (176.3, 13.1)
- added D64: WS2812B, LED_SMD:LED_WS2812B_PLCC4_5.0x5.0mm_P3.2mm, B.Cu at (204.6, 13.1)
- added D65: WS2812B, LED_SMD:LED_WS2812B_PLCC4_5.0x5.0mm_P3.2mm, B.Cu at (227.6, 13.0)
- added D66: WS2812B, LED_SMD:LED_WS2812B_PLCC4_5.0x5.0mm_P3.2mm, B.Cu at (251.8, 13.1)
Connections:
- U1 pad 29: unconnected-(U1-GPIO22-Pad29) -> Data in LED
- U1 pad 38: unconnected-(U1-GND-Pad38) -> GND
- U1 pad 40: unconnected-(U1-VBUS-Pad40) -> 5V
Routing:
- net Data in LED: track 0.00 -> 277.2 mm, vias 0 -> 3
- net GND: track 0.00 -> 252.3 mm
- net 5V: track 0.00 -> 245.8 mm
- net col13: track 126.3 -> 166.0 mm
- net Net-(D59-DOUT): track 0.00 -> 24.8 mm
- net Net-(D44-DOUT): track 0.00 -> 23.7 mm
- net Net-(D29-DOUT): track 0.00 -> 22.2 mm
- net Net-(D47-DOUT): track 0.00 -> 21.0 mm
- net Net-(D32-DOUT): track 0.00 -> 21.0 mm
- net Net-(D65-DOUT): track 0.00 -> 20.6 mm
- net Net-(D14-DOUT): track 0.00 -> 20.4 mm
- net Net-(D64-DOUT): track 0.00 -> 19.6 mm
- net Net-(D17-DOUT): track 0.00 -> 16.7 mm
- net col2: track 319.1 -> 335.3 mm, vias 1 -> 2
- net col3: track 270.8 -> 287.0 mm, vias 3 -> 4
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
Commit message: rebuilding gbr files and pcb for better soldering ease
Parts:
- D1, D10, D11, D12, D120, D121, D13, D15, D16, D18, D19, D2, D20, D21, D22, D23, D24, D25, D26, D27, D28, D3, D30, D31, D33, D34, D35, D36, D37, D38, D39, D4, D40, D41, D42, D43, D45, D46, D48, D49, D5, D50, D51, D52, D53, D54, D55, D56, D57, D58, D6, D60, D61, D62, D63, D68, D7, D73, D74, D75, D8, D9: footprint Diode_SMD:D_SOD-123F -> ScottoKeebs_Components:Diode_DO-35
- D14, D17, D29, D32, D44, D47, D59, D64, D65, D66, G***: moved to F.Cu
- moved D75 29.8 mm to (263.8, 124.4)
- moved D58 29.5 mm to (227.3, 106.9)
- moved D68 29.2 mm to (207.8, 123.7)
- moved D74 28.2 mm to (244.8, 124.3)
- moved D63 27.9 mm to (65.5, 123.5)
- moved D60 27.8 mm to (247.9, 106.4)
- moved D121 27.7 mm to (86.3, 123.6)
- moved D53 27.5 mm to (136.7, 107.8)
- moved D35 27.5 mm to (82.9, 89.4)
- moved D54 27.4 mm to (154.9, 107.0)
- moved D21 27.4 mm to (100.9, 72.1)
- moved D30 27.4 mm to (263.1, 72.4)
- moved D73 27.3 mm to (227.1, 123.7)
- moved D56 27.3 mm to (191.1, 106.8)
- moved D19 27.3 mm to (65.1, 72.2)
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Connections:
- S17 pad 1: row3 -> col9
- S29 pad 1: row3 -> col4
Routing:
- net col12: track 238.6 -> 155.0 mm, vias 8 -> 2
- net col7: track 277.2 -> 215.8 mm
- net row3: track 334.7 -> 276.4 mm, vias 2 -> 0
- net col13: track 166.0 -> 117.8 mm, vias 4 -> 2
- net col4: track 353.5 -> 309.8 mm
- net col5: track 305.6 -> 275.0 mm
- net unconnected-(U1-GND-Pad13): track 30.1 -> 0.00 mm
- net row0: track 298.7 -> 270.1 mm, vias 28 -> 3
- net col9: track 200.0 -> 227.6 mm, vias 7 -> 2
- net row1: track 262.2 -> 243.9 mm, vias 32 -> 1
- net col8: track 216.0 -> 233.2 mm
- net col11: track 171.3 -> 154.7 mm, vias 5 -> 2
- net col14: track 151.5 -> 138.1 mm, vias 4 -> 0
- net row2: track 266.0 -> 252.9 mm, vias 26 -> 0
- net col1: track 340.9 -> 330.5 mm, vias 2 -> 0
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Other:
- board size 299.8 x 97 mm -> 297.5 x 97.7 mm
